File: _autosave-matrix_board.kicad_pcb (KiCad board)
At the start: 2 copper layers, 68.1 x 40.1 mm, 10 parts, among them J1 MATRIX_CONNECTOR, M1 PWR_LED, M2 LED, U1 ATmega328P-AU

Commit message: remade board to be bigger
Parts:
- added M3: PINHD-2X2-SMD, fab:fab-2X02SMD, F.Cu at (162.1, 53.3)
Routing:
- net VCC: track 115.1 -> 150.3 mm
- net GROUND: track 245.3 -> 264.3 mm
- net A: track 52.7 -> 59.1 mm
- net C: track 53.9 -> 50.8 mm
- net RESET: track 35.6 -> 38.4 mm
- net LAT: track 46.4 -> 47.1 mm
Other:
- net class Default: clearance 0.3 -> 0.4
- rule trace_clearance: 0.3 -> 0.4

Commit message: updated board with more components so it'll work
added pull up resistor on reset and clock on xtal, also moved capacitor closer to chip
Parts:
- added M4: RESONATOR, fab:fab-EFOBM, F.Cu at (146.7, 75.6)
- added R3: 10k, fab:fab-R1206, F.Cu at (156.3, 60.2)
- J1: footprint Connector_PinHeader_2.00mm:PinHeader_2x08_P2.00mm_Vertical_SMD -> fab:fab-2X08SMD
- moved C1 13.2 mm to (166.6, 74.5), turned to 270 degrees
- moved J1 7.20 mm to (131.9, 65.0)
Connections:
- U1 pad 7: Net-(U1-Pad7) -> XTAL1
- U1 pad 8: Net-(U1-Pad8) -> XTAL2
Routing:
- net GROUND: track 264.3 -> 273.8 mm
- net XTAL1: track 0.00 -> 9.07 mm
- net XTAL2: track 0.00 -> 8.35 mm
- net VCC: track 150.3 -> 156.2 mm
- net R2: track 30.0 -> 35.7 mm
- net B2: track 32.8 -> 37.4 mm
- net G2: track 27.3 -> 31.2 mm
- net PD1: track 34.4 -> 30.7 mm
- net RESET: track 38.4 -> 42.0 mm
- net CLK: track 31.1 -> 33.9 mm
- net R1: track 28.0 -> 30.4 mm
- net B1: track 26.7 -> 28.9 mm
- net D: track 38.3 -> 36.6 mm
- net SCK: track 25.3 -> 26.6 mm
- net A: track 59.1 -> 57.8 mm
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